Commit message: Future | Multi car racing setup - Fixed glitching error

File: base_system/f110-simulator/racecar.xacro (robot description, xacro)
@@ -2,4 +2,7 @@
 <!-- A simple model of the racecar for rviz -->
 <robot xmlns:xacro="http://www.ros.org/wiki/xacro" name="racecar">
+  <!-- Frame prefix parameter for multi-car support -->
+  <xacro:arg name="frame_prefix" default=""/>
+  <xacro:property name="frame_prefix" value="$(arg frame_prefix)"/>
   <xacro:property name="wheelbase" value="0.3302" />
   <xacro:property name="width" value="0.2032" />
@@ -17,5 +20,5 @@
     <color rgba="0.3 0.57 1. 1."/>
   </material>
-  <link name="base_link">
+  <link name="${frame_prefix}base_link">
     <visual>
       <origin xyz="${wheelbase/2} 0 ${ground_offset+height/2}"/>
@@ -26,10 +29,10 @@
     </visual>
   </link>
-  <joint name="base_to_laser_model" type="fixed">
-    <parent link="base_link"/>
-    <child link="laser_model"/>
+  <joint name="${frame_prefix}base_to_laser_model" type="fixed">
+    <parent link="${frame_prefix}base_link"/>
+    <child link="${frame_prefix}laser_model"/>
     <origin xyz="${laser_distance_from_base_link} 0 ${ground_offset+height+(laser_height/2)}"/>
   </joint>
-  <link name="laser_model">
+  <link name="${frame_prefix}laser_model">
     <visual>
       <geometry>
@@ -40,9 +43,9 @@
   </link>
   <joint name="base_to_back_left_wheel" type="fixed">
-    <parent link="base_link"/>
-    <child link="back_left_wheel"/>
+    <parent link="${frame_prefix}base_link"/>
+    <child link="${frame_prefix}back_left_wheel"/>
     <origin xyz="0 ${(wheel_length+width)/2} ${wheel_radius}"/>
   </joint>
-  <link name="back_left_wheel">
+  <link name="${frame_prefix}back_left_wheel">
     <visual>
       <geometry>
@@ -54,9 +57,9 @@
   </link>
   <joint name="base_to_back_right_wheel" type="fixed">
-    <parent link="base_link"/>
-    <child link="back_right_wheel"/>
+    <parent link="${frame_prefix}base_link"/>
+    <child link="${frame_prefix}back_right_wheel"/>
     <origin xyz="0 ${-(wheel_length+width)/2} ${wheel_radius}"/>
   </joint>
-  <link name="back_right_wheel">
+  <link name="${frame_prefix}back_right_wheel">
     <visual>
       <geometry>
@@ -68,14 +71,14 @@
   </link>
   <joint name="base_to_front_left_hinge" type="fixed">
-    <parent link="base_link"/>
-    <child link="front_left_hinge"/>
+    <parent link="${frame_prefix}base_link"/>
+    <child link="${frame_prefix}front_left_hinge"/>
     <origin xyz="${wheelbase} ${(wheel_length+width)/2} ${wheel_radius}"/>
   </joint>
-  <link name="front_left_hinge"/>
-  <joint name="front_left_hinge_to_wheel" type="continuous">
-    <parent link="front_left_hinge"/>
-    <child link="front_left_wheel"/>
+  <link name="${frame_prefix}front_left_hinge"/>
+  <joint name="front_left_hinge_to_wheel" type="fixed">
+    <parent link="${frame_prefix}front_left_hinge"/>
+    <child link="${frame_prefix}front_left_wheel"/>
   </joint>
-  <link name="front_left_wheel">
+  <link name="${frame_prefix}front_left_wheel">
     <visual>
       <geometry>
@@ -87,14 +90,14 @@
   </link>
   <joint name="base_to_front_right_hinge" type="fixed">
-    <parent link="base_link"/>
-    <child link="front_right_hinge"/>
+    <parent link="${frame_prefix}base_link"/>
+    <child link="${frame_prefix}front_right_hinge"/>
     <origin xyz="${wheelbase} ${-(wheel_length+width)/2} ${wheel_radius}"/>
   </joint>
-  <link name="front_right_hinge"/>
-  <joint name="front_right_hinge_to_wheel" type="continuous">
-    <parent link="front_right_hinge"/>
-    <child link="front_right_wheel"/>
+  <link name="${frame_prefix}front_right_hinge"/>
+  <joint name="front_right_hinge_to_wheel" type="fixed">
+    <parent link="${frame_prefix}front_right_hinge"/>
+    <child link="${frame_prefix}front_right_wheel"/>
   </joint>
-  <link name="front_right_wheel">
+  <link name="${frame_prefix}front_right_wheel">
     <visual>
       <geometry>
